Commit message: turretモデルの追加

File: urdf/proto1.xacro (robot description, xacro)
@@ -3,4 +3,6 @@
   <xacro:include filename="$(find attracts_description)/urdf/mobile_base.xacro" />
   <xacro:include filename="$(find attracts_description)/urdf/wheel.xacro" />
+  <xacro:include filename="$(find attracts_description)/urdf/turret_base.xacro" />
+  <xacro:include filename="$(find attracts_description)/urdf/turret_unit.xacro" />
   <xacro:mobile_base />
   <xacro:wheel prefix="right" suffix="front" />
@@ -32,3 +34,18 @@
     <origin xyz="-0.0880347 0.0880347 0.03" rpy="${pi/2} 0 ${-3*pi/4}" />
   </joint>
+  <xacro:turret_base />
+  <joint name="yaw_joint" type="continuous">
+    <parent link="base_link" />
+    <child link="yaw_link" />
+    <axis xyz="0 0 1" />
+    <origin xyz="0.0 0.0 0.124" rpy="0 0 0" />
+  </joint>
+  <xacro:turret_unit />
+  <joint name="pitch_joint" type="revolute">
+    <parent link="yaw_link" />
+    <child link="pitch_link" />
+    <axis xyz="0 0 1" />
+    <origin xyz="-0.03 -0.0466 0.042" rpy="${pi/2} 0 0" />
+    <limit lower="${-pi/12}" upper="${pi/6}" effort="0" velocity="0"/>
+  </joint>
 </robot>
